File: Esquematico+BOM/Esquematico_Encoder.sch (EAGLE design)
At the start: 11 parts

Commit message: Se agregaron archivos de la entrega de PCB
Connections:
- net GND: no longer M1-CN6.RESET, M1-CN7.RESET
Changed lines of the file:
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@@
 <part name="GND12" library="supply1" library_urn="urn:adsk.eagle:library:371" deviceset="GND" device=""/>
 <part name="GND13" library="supply1" library_urn="urn:adsk.eagle:library:371" deviceset="GND" device=""/>
-<part name="GND14" library="supply1" library_urn="urn:adsk.eagle:library:371" deviceset="GND" device=""/>
 </parts>
 <sheets>
@@
 <attribute name="VALUE" x="-22.86" y="-106.68" size="1.778" layer="96"/>
 </instance>
-<instance part="GND14" gate="1" x="15.24" y="-45.72" smashed="yes" rot="R180">
-<attribute name="VALUE" x="17.78" y="-43.18" size="1.778" layer="96" rot="R180"/>
-</instance>
 </instances>
 <busses>
@@
 <pinref part="M1" gate="-CN7" pin="GND@2"/>
 <wire x1="-99.06" y1="-60.96" x2="-93.98" y2="-60.96" width="0.1524" layer="91"/>
-<wire x1="-93.98" y1="-60.96" x2="-93.98" y2="-68.58" width="0.1524" layer="91"/>
-<pinref part="M1" gate="-CN7" pin="RESET"/>
-<wire x1="-93.98" y1="-68.58" x2="-93.98" y2="-76.2" width="0.1524" layer="91"/>
-<wire x1="-99.06" y1="-68.58" x2="-93.98" y2="-68.58" width="0.1524" layer="91"/>
-<junction x="-93.98" y="-68.58"/>
+<wire x1="-93.98" y1="-60.96" x2="-93.98" y2="-76.2" width="0.1524" layer="91"/>
 </segment>
 <segment>
@@
 <wire x1="-20.32" y1="-73.66" x2="-20.32" y2="-101.6" width="0.1524" layer="91"/>
 </segment>
-<segment>
-<pinref part="M1" gate="-CN6" pin="RESET"/>
-<pinref part="GND14" gate="1" pin="GND"/>
-<wire x1="20.32" y1="-53.34" x2="15.24" y2="-53.34" width="0.1524" layer="91"/>
-<wire x1="15.24" y1="-53.34" x2="15.24" y2="-48.26" width="0.1524" layer="91"/>
-</segment>
-</net>
+</net>
